File: Electrical hardware/LCMscope.kicad_pcb (KiCad board)
At the start: 2 copper layers, 6 parts, among them U1 ICE40UP5K-SG48ITR, U2 LTC2299xUP, U3 MIC5365-3.3YC5, U4 TLV70212_SOT23-5, U5 TLV73325PDBV, Y1 ASV-xxxMHz

Commit message: Created ADC footprint and extracted most important data from the data sheet
Parts:
- U2: value LTC2299xUP -> LTC2254; footprint Package_DFN_QFN:QFN-64-1EP_9x9mm_P0.5mm_EP7.15x7.15mm -> Package_DFN_QFN:QFN-32-1EP_5x5mm_P0.5mm_EP3.45x3.45mm
- moved U2 12.1 mm to (79.7, 42.3)
Connections:
- U2 pad 1: unconnected-(U2-AINA+-Pad1) -> /ADC/V+
- U2 pad 11: Net-(U2-REFLB-Pad11) -> unconnected-(U2-OE-Pad11)
- U2 pad 12: Net-(U2-REFLB-Pad11) -> unconnected-(U2-D0_LSB-Pad12)
- U2 pad 13: Net-(U2-REFHB-Pad13) -> unconnected-(U2-D1-Pad13)
- U2 pad 14: Net-(U2-REFHB-Pad13) -> unconnected-(U2-D2-Pad14)
- U2 pad 17: Net-(U2-GND-Pad17) -> Net-(U2-D5)
- U2 pad 18: unconnected-(U2-VDD-Pad18) -> Net-(U2-D5)
- U2 pad 2: unconnected-(U2-AINA--Pad2) -> /ADC/V-
- U2 pad 3: Net-(U2-REFHA-Pad3) -> unconnected-(U2-REFH-Pad3)
- U2 pad 31: Net-(U2-OGND-Pad31) -> unconnected-(U2-VCM-Pad31)
- U2 pad 4: Net-(U2-REFHA-Pad3) -> unconnected-(U2-REFH-Pad4)
- U2 pad 5: Net-(U2-REFLA-Pad5) -> unconnected-(U2-REFL-Pad5)
- U2 pad 6: Net-(U2-REFLA-Pad5) -> unconnected-(U2-REFL-Pad6)
